File: board/TOFE-HiLink.sch (KiCad schematic (older format))
At the start: 6 parts, among them U1 TOFE-8X, U7 24AA01/24LC01B

Commit message: Slowly figuring things out.
Parts:
- added J? (x3): DISPLAY_PORT, symbol DISPLAY_PORT
- added J?: DISPLAY_PORT_SRC, symbol DISPLAY_PORT_SRC
- added J?: DISPLAY_PORT_SINK, symbol DISPLAY_PORT_SINK
Connections:
- net labels added: DP_RX1_IO0, DP_RX1_N0, DP_RX1_N1, DP_RX1_N2, DP_RX1_N3, DP_RX1_N4, DP_RX1_P0, DP_RX1_P1, DP_RX1_P2, DP_RX1_P3, DP_RX1_P4, DP_RX1_SCL, DP_RX1_SDA, DP_TX1_IO0, DP_TX1_N0, DP_TX1_N1, DP_TX1_N2, DP_TX1_N3, DP_TX1_N4, DP_TX1_N[0..4], DP_TX1_P0, DP_TX1_P1, DP_TX1_P2, DP_TX1_P3, DP_TX1_P4, DP_TX1_P[0..4], DP_TX1_SCL, DP_TX1_SDA, SCL_REMOTE_N, SCL_REMOTE_S, SDA_REMOTE_N, SDA_REMOTE_S
- wire segments 79 -> 204
